Commit message: URDF completed revH and readme added

File: mh5_description/urdf/mh5_leg_revH.xacro (robot description, xacro)
@@ -198,5 +198,5 @@
                 <origin rpy="0 0 0" xyz="0 0 0"/>
                 <geometry>
-                    <mesh filename="package://mh5_description/meshes/foot_${side}_revE.stl"/>
+                    <mesh filename="package://mh5_description/meshes/foot_revH.dae"/>
                 </geometry>
                 <xacro:material_ivory/>
@@ -205,25 +205,25 @@
                 <origin rpy="0 0 0" xyz="0 0 0"/>
                 <geometry>
-                    <mesh filename="package://mh5_description/meshes/foot_${side}_revE.stl"/>
-                </geometry>
-            </collision>
-            <inertial>
-                <origin rpy="0 0 0" xyz="0 0 0"/>
-                <mass value="0.053"/>
-                <inertia
-                    ixx="0.000027639"
-                    iyy="0.000067044"
-                    izz="0.000083497"
-                    ixy="-0.000000056"
-                    ixz="0.000001332"
-                    iyz="0.0000000012" />
-            </inertial>
-        </link>
-        <joint name="${side}_battery_fixed" type="fixed">
+                    <mesh filename="package://mh5_description/meshes/foot_revH.dae"/>
+                </geometry>
+            </collision>
+            <inertial>
+                <origin rpy="0 0 0" xyz="0 0 0"/>
+                <mass value="0.038"/>
+                <inertia
+                    ixx="0.000006451"
+                    iyy="0.000022262"
+                    izz="0.000026598"
+                    ixy="0.000000000"
+                    ixz="0.000000341"
+                    iyz="0.000000000" />
+            </inertial>
+        </link>
+        <!-- <joint name="${side}_battery_fixed" type="fixed">
             <parent link="${side}_foot"/>
             <child link="${side}_battery"/>
             <origin xyz="0.015 ${factor*0.009} -0.037" rpy="0 0 0"/>
-        </joint>
-        <link name="${side}_battery">
+        </joint> -->
+        <!-- <link name="${side}_battery">
             <visual>
                 <origin rpy="0 0 0" xyz="0 0 0"/>
@@ -252,11 +252,11 @@
                     iyz="0.000000000" />
             </inertial>
-        </link>
-        <joint name="${side}_sole_fixed" type="fixed">
+        </link> -->
+        <!-- <joint name="${side}_sole_fixed" type="fixed">
             <parent link="${side}_foot"/>
             <child link="${side}_landing"/>
             <origin xyz="0.0 0.0 -0.03825" rpy="0 0 0"/>
-        </joint>
-        <link name="${side}_landing" />
+        </joint> -->
+        <!-- <link name="${side}_landing" /> -->
     </xacro:macro>
 </robot>

File: mh5_description/urdf/mh5_robot_revH.urdf.xacro (robot description, xacro)
@@ -1,10 +1,11 @@
 <?xml version="1.0" ?>
 <robot xmlns:xacro="http://ros.org/wiki/xacro" name="mh5_robot">
+    <xacro:include filename="$(find mh5_description)/urdf/mh5_chest_revH.xacro"/>
     <xacro:include filename="$(find mh5_description)/urdf/mh5_head_revH.xacro"/>
     <xacro:include filename="$(find mh5_description)/urdf/mh5_arm_revH.xacro"/>
-    <!-- <xacro:include filename="$(find mh5_description)/urdf/mh5_leg_revE.xacro"/> -->
+    <xacro:include filename="$(find mh5_description)/urdf/mh5_leg_revH.xacro"/>
     <xacro:macro name="material_ivory">
         <material name="ivory">
-            <color rgba="1 1 0.94 1"/>
+            <color rgba="0.8 0.8 0.8 1"/>
         </material>
     </xacro:macro>
@@ -15,39 +16,10 @@
     </xacro:macro>
     <link name="base_link"/>
-    <link name="chest">
-        <visual>
-            <origin rpy="0 0 0" xyz="0 0 0"/>
-            <geometry>
-                <mesh filename="package://mh5_description/meshes/chest_revH.dae"/>
-            </geometry>
-            <xacro:material_ivory/>
-        </visual>
-        <collision>
-            <origin rpy="0 0 0" xyz="0 0 0"/>
-            <geometry>
-                <mesh filename="package://mh5_description/meshes/chest_revH.dae"/>
-            </geometry>
-        </collision>
-        <inertial>
-            <mass value="0.400"/>
-            <inertia
-                ixx="0.000954830"
-                iyy="0.000597536"
-                izz="0.000637274"
-                ixy="-0.000001668"
-                ixz="-0.000021416"
-                iyz="0.000000148" />
-        </inertial>
-    </link>
-    <joint name="chest_fixed" type="fixed">
-        <parent link="base_link"/>
-        <child link="chest"/>
-        <origin xyz="0 0 0.203" rpy="0 0 0"/>
-    </joint>
+    <xacro:mh5_chest parent="base_link" />
     <xacro:mh5_head parent="chest" />
     <xacro:mh5_arm side="left" parent="chest" />
     <xacro:mh5_arm side="right" parent="chest" />
-    <!-- <xacro:mh5_leg side="left" parent="chest" />
-    <xacro:mh5_leg side="right" parent="chest" /> -->
+    <xacro:mh5_leg side="left" parent="chest" />
+    <xacro:mh5_leg side="right" parent="chest" />
     <gazebo>
         <plugin name="gazebo_ros_control" filename="libgazebo_ros_control.so">
