Commit message: rev H plus fix for head collision orientation

File: mh5_description/urdf/mh5_chest_revH.xacro (robot description, xacro)
@@ -27,5 +27,5 @@
             </inertial>
         </link>
-        <joint name="chest_fixed" type="fixed">
+        <joint name="chest_fixed" type="floating">
             <parent link="${parent}"/>
             <child link="chest"/>

File: mh5_description/urdf/mh5_head_revH.xacro (robot description, xacro)
@@ -20,5 +20,5 @@
             </visual>
             <collision>
-                <origin rpy="0 0 0" xyz="0 0 0"/>
+                <origin rpy="0 ${pi/2} ${pi}" xyz="0 0 0"/>
                 <geometry>
                     <mesh filename="package://mh5_description/meshes/2XL430_1_idle_revC.stl"/>
